Commit message: "Debug quality"

File: cart_pole_description/cart_pole/robot.urdf (robot description, URDF)
Before this commit: robot cart_pole, 5 links, 4 joints
Links:
- added link world
Joints:
- added joint world_to_base_joint: type fixed, parent world, child support_pole, origin xyz=0.0 0.0 0.0 rpy=0.0 0.0 0.0

Commit message: "added the gazebo"

File: cart_pole_description/cart_pole/robot.urdf (robot description, URDF)
Before this commit: robot cart_pole, 6 links, 5 joints
Links:
- removed link world
Joints:
- removed joint world_to_base_joint
