Commit message: "succeffully set up the effort control"

File: cart_pole_description/cart_pole/ros2_control.urdf.xacro (robot description, xacro)
@@ -1,29 +1,24 @@
 <?xml version="1.0"?>
 <robot xmlns:xacro="http://www.ros.org/wiki/xacro">
-    <ros2_control name="gazebo_control" type="system">
-        <hardware>
-            <plugin>gazebo_ros2_control/GazeboSystem</plugin>
-        </hardware>
-        <joint name="slider_1">
-            <command_interface name="position">
-                <param name="min">-1.57</param>
-                <param name="max">1.57</param>
-            </command_interface>
-            <command_interface name="velocity">
-                <param name="min">-100</param>
-                <param name="max">100</param>
-            </command_interface>
-            <state_interface name="position">
-                <param name="initial_value">0.0</param>
-            </state_interface>
-            <state_interface name="velocity"/>
-        </joint>
-    </ros2_control>
-    <gazebo>
-        <plugin filename="libgazebo_ros2_control.so" name="gazebo_ros2_control">
-           <robot_param>robot_description</robot_param>
-           <robot_param_node>robot_state_publisher</robot_param_node>
-           <parameters>$(find cart_pole_description)/config/effort_control.yaml</parameters>
-        </plugin>
-    </gazebo>
+<ros2_control name="GazeboSimSystem" type="system">
+  <hardware>
+    <plugin>gazebo_ros2_control/GazeboSystem</plugin>
+  </hardware>
+  <joint name="slider_1">
+    <command_interface name="effort">
+      <param name="min">-1000</param>
+      <param name="max">1000</param>
+    </command_interface>
+    <state_interface name="position">
+      <param name="initial_value">1.0</param>
+    </state_interface>
+    <state_interface name="velocity"/>
+    <state_interface name="effort"/>
+  </joint>
+</ros2_control>
+  <gazebo>
+    <plugin filename="libgazebo_ros2_control.so" name="gazebo_ros2_control">
+      <parameters>$(find cart_pole_description)/config/effort_control.yaml</parameters>
+    </plugin>
+  </gazebo>
 </robot>
