Commit message: "with gazebo launch and ros2 control, at this point the forward_mmand controller does not work with it."

File: cart_pole_description/cart_pole/robot.urdf.xacro (robot description, xacro)
@@ -1,3 +1,5 @@
-<robot name="cart_pole">
+<?xml version="1.0"?>
+<robot name="cart_pole" xmlns:xacro="http://wiki.ros.org/xacro">
+<xacro:include filename="$(find cart_pole_description)/cart_pole/ros2_control.urdf.xacro"/>
 <link name="support_pole">
 <visual>
@@ -126,5 +128,5 @@
 <joint_properties friction="0.0"/>
 </joint>
-<joint name="slider 1" type="prismatic">
+<joint name="slider_1" type="prismatic">
 <origin xyz="-0.99499999999999999556 -0.024999999999999966693 0.040000000000000035527" rpy="-0 -1.570796326794896558 0" />
 <parent link="cart_pole" />

Commit message: "added the reading of state interfaces fos the position of the pendulum and cart"

File: cart_pole_description/cart_pole/robot.urdf.xacro (robot description, xacro)
@@ -120,5 +120,5 @@
 </inertial>
 </link>
-<joint name="continuous_revolute 1" type="continuous">
+<joint name="continuous_revolute_1" type="continuous">
 <origin xyz="0.035000000000000003331 0.024999999999999966693 0" rpy="-0 -1.570796326794896336 0" />
 <parent link="cart_move" />

File: cart_pole_description/cart_pole/ros2_control.urdf.xacro (robot description, xacro)
@@ -16,4 +16,11 @@
     <state_interface name="effort"/>
   </joint>
+  <joint name="continuous_revolute_1">
+     <!-- leaving it empty because I am that good-->
+    <state_interface name="position">
+       <param name="initial_value">0.0</param>
+       </state_interface>
+    <state_interface name="velocity"/>
+  </joint>
 </ros2_control>
   <gazebo>

Commit message: "controller works great, but hits the pole too soone, maybe I should give it more space"

File: cart_pole_description/cart_pole/robot.urdf.xacro (robot description, xacro)
@@ -125,5 +125,5 @@
 <child link="cart_swinger" />
 <axis xyz="0 0 1"/>
-<limit effort="1" velocity="20" />
+<limit effort="1" velocity="30" />
 <joint_properties friction="0.0"/>
 </joint>
@@ -133,5 +133,5 @@
 <child link="cart_move" />
 <axis xyz="0 0 1"/>
-<limit effort="1" velocity="20" lower="-0.8499999999999999778" upper="0.8499999999999999778"/>
+<limit effort="500" velocity="30" lower="-0.8499999999999999778" upper="0.8499999999999999778"/>
 <joint_properties friction="0.0"/>
 </joint>
